File: clonos.brd (EAGLE design)
At the start: 67 x 110 mm, 120 parts, among them J1 POWER_JACKPTH, Q1 HC49/S1, T1 BC846B, T2 BC846B, U1 MCIMX233CAG4C, U2 HY5DU121622D(L)T(P)-J, U5 MP1482DS, U6 SY8008C(AA)C

Commit message: Some work on the schematic
Connections:
- net PIN1/LCD_D00 renamed BOOT1
- net PIN2/LCD_D01 renamed BOOT2
- net PIN25/LCD_RS renamed BOOT
- net PIN3/LCD_D02 renamed BOOT3
- net PIN4/LCD_D03 renamed BOOT4
- net PIN6/LCD_D05 renamed ETM
Changed lines of the file:
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@@
 <wire x1="40.028" y1="90.889" x2="41.238" y2="68.718" width="0" layer="19" extent="1-1"/>
 </signal>
-<signal name="PIN1/LCD_D00">
-<contactref element="U1" pad="2"/>
-<contactref element="RM3" pad="4.1"/>
-<contactref element="RM2" pad="4.2"/>
-<wire x1="31.6128" y1="61.99" x2="33.848" y2="61.99" width="0" layer="19" extent="1-1"/>
-<wire x1="37.6" y1="55.13" x2="31.6128" y2="61.99" width="0" layer="19" extent="1-1"/>
-</signal>
-<signal name="PIN2/LCD_D01">
+<signal name="BOOT2">
 <contactref element="U1" pad="3"/>
 <contactref element="RM3" pad="3.1"/>
@@
 <wire x1="37.2" y1="55.13" x2="31.6128" y2="61.101" width="0" layer="19" extent="1-1"/>
 </signal>
-<signal name="PIN3/LCD_D02">
+<signal name="BOOT3">
 <contactref element="U1" pad="4"/>
 <contactref element="RM3" pad="2.1"/>
@@
 <wire x1="36.8" y1="55.13" x2="31.6128" y2="60.339" width="0" layer="19" extent="1-1"/>
 </signal>
-<signal name="PIN4/LCD_D03">
+<signal name="BOOT4">
 <contactref element="U1" pad="5"/>
 <contactref element="RM3" pad="1.1"/>
@@
 <wire x1="36.4" y1="55.13" x2="31.6128" y2="59.45" width="0" layer="19" extent="1-1"/>
 </signal>
-<signal name="PIN6/LCD_D05">
+<signal name="ETM">
 <contactref element="U1" pad="7"/>
 <contactref element="R14" pad="2"/>
@@
 <wire x1="35.2" y1="39.63" x2="43.011" y2="94.831" width="0" layer="19" extent="1-1"/>
 </signal>
-<signal name="PIN25/LCD_RS">
+<signal name="BOOT">
 <contactref element="U1" pad="14"/>
 <contactref element="R15" pad="2"/>
@@
 <contactref element="U1" pad="100"/>
 </signal>
+<signal name="BOOT1">
+<contactref element="RM3" pad="4.1"/>
+<contactref element="RM2" pad="4.2"/>
+<contactref element="U1" pad="2"/>
+<wire x1="31.6128" y1="61.99" x2="33.848" y2="61.99" width="0" layer="19" extent="1-1"/>
+<wire x1="37.6" y1="55.13" x2="33.848" y2="61.99" width="0" layer="19" extent="1-1"/>
+</signal>
 </signals>

Commit message: Audio switching
Parts:
- removed U$3, U$4, U$6: A5W-K, clonos:A5W-K
- added D1, D2, D5: 1N4148, adafruit:SOD-323F
- added FB1, FB2, FB3, FB4, FB5, FB6: HZ0805D152R, dp_devices:FB805
- added R11: 1k, rcl:R0603_5MIL_DWS
- added REL1, REL2, REL3: A5W-K-BIS, clonos:A5W-K
- added T3, T4, T5: BC846B, semicon-smd-ipc:SOT23
Connections:
- new net N$13: FB1.1, HEADPHONES.3
- new net N$15: FB2.1, HEADPHONES.2
- new net N$16: FB3.1, HEADPHONES.5
- new net N$17: FB5.1, LINE_IN.2
- new net N$20: FB4.1, LINE_IN.3
- new net N$21: FB6.1, LINE_IN.5
- new net N$22: D1.A, REL1.COIL-, T3.3
- new net N$23: R11.1
- new net N$24: D2.A, REL2.COIL-, T4.3
- new net N$26: R11.2, T3.1, T4.1, T5.1
- new net N$29: D5.A, REL3.COIL-, T5.3
- net +5V: now also D1.C, D2.C, D5.C, REL1.COIL+, REL2.COIL+, REL3.COIL+
- net GND: now also REL1.COM2, T3.2, T4.2, T5.2; no longer U$3.COM2
- net HPL: now also REL2.COM2; no longer U$4.COM2
- net HPR: now also REL2.COM1; no longer U$4.COM1
- net HP_VGND: now also REL1.NO1; no longer U$3.NO1
- net N$11: now also FB4.2, REL3.COM1; no longer LINE_IN.3, U$6.COM1
- net N$12: now also FB3.2, REL1.COM1; no longer HEADPHONES.5, U$3.COM1
- net N$14: now also FB6.2, REL1.NC1, REL1.NO2; no longer LINE_IN.5, U$3.NC1, U$3.NO2
- net N$2: now also REL3.NO1; no longer U$6.NO1
- net N$3: now also FB1.2, REL2.NO1, REL3.NC1; no longer HEADPHONES.3, U$4.NO1, U$6.NC1
- net N$4: now also FB2.2, REL2.NO2, REL3.NC2; no longer HEADPHONES.2, U$4.NO2, U$6.NC2
- net N$5: now also FB5.2, REL3.COM2; no longer LINE_IN.2, U$6.COM2
- net N$6: now also REL3.NO2; no longer U$6.NO2
