File: clonos.sch (EAGLE design)
At the start: 117 parts, among them J1 POWER_JACKPTH, Q1 HC49/S1, T1 BC846B, T2 BC846B, U1 MCIMX233CAG4C, U2 HY5DU121622D(L)T(P)-J, U5 MP1482DS, U6 SY8008C(AA)C

Commit message: Some work on the schematic
Connections:
- net PIN1/LCD_D00 renamed BOOT1
- net PIN2/LCD_D01 renamed BOOT2
- net PIN25/LCD_RS renamed BOOT
- net PIN3/LCD_D02 renamed BOOT3
- net PIN4/LCD_D03 renamed BOOT4
- net PIN6/LCD_D05 renamed ETM
Other:
- note added: "Boot mode"
- note removed: "0"
- note removed: "1"
- note removed: "3.3V I2C Master"
- note removed: "3.3V NAND"
- note removed: "3.3V SD/MMC 1 (Default !!!)"
- note removed: "3.3V SD/MMC 2"
- note removed: "3.3V SPI Flash 1 Master"
- note removed: "3.3V SPI Flash 2 Master"
- note removed: "BOOT MODE"
- note removed: "BOOT MODE SELECT"
- note removed: "BOOT MODE SELECT:"
- note removed: "D00"
- note removed: "D01"
- note removed: "D02"
- note removed: "D03"
- note removed: "High to enable Resistor Boot Mode."
- note removed: "If pulled low, the i.MX233 will"
- note removed: "LCD DATA"
- note removed: "LCD_RS must to be pulled"
- note removed: "Startup waits for JTAG debugger connection"
- note removed: "attempt to boot from OTP."
- moved on the sheet: C68, C69, C70, C71, C72, C73, C74, C75, C79, C80, D3, J1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

Commit message: Audio switching
Parts:
- removed U$3, U$4, U$6: A5W-K, clonos:A5W-K
- added D1, D2, D5: 1N4148, adafruit:DIODESOD-323F
- added FB1, FB2, FB3, FB4, FB5, FB6: HZ0805D152R, dp_devices:FERRITE-0805
- added R11: 1k, rcl:R-EU_R0603_5MIL_DWS
- added REL1, REL2, REL3: A5W-K-BIS, clonos:A5W-K-BIS
- added T3, T4, T5: BC846B, semicon-smd-ipc:NPN-TRANSISTOR_SOT23
Connections:
- new net N$13: FB1.1, HEADPHONES.3
- new net N$15: FB2.1, HEADPHONES.2
- new net N$16: FB3.1, HEADPHONES.5
- new net N$17: FB5.1, LINE_IN.2
- new net N$20: FB4.1, LINE_IN.3
- new net N$21: FB6.1, LINE_IN.5
- new net N$22: D1.A, REL1COIL.COIL-, T3.C
- new net N$23: R11.1
- new net N$24: D2.A, REL2COIL.COIL-, T4.C
- new net N$26: R11.2, T3.B, T4.B, T5.B
- new net N$29: D5.A, REL3COIL.COIL-, T5.C
- net +5V: now also D1.C, D2.C, D5.C, REL1COIL.COIL+, REL2COIL.COIL+, REL3COIL.COIL+
- net GND: now also REL1B.COM, T3.E, T4.E, T5.E; no longer U$3.COM2
- net HPL: now also REL2B.COM; no longer U$4.COM2
- net HPR: now also REL2A.COM; no longer U$4.COM1
- net HP_VGND: now also REL1A.NO; no longer U$3.NO1
- net N$11: now also FB4.2, REL3A.COM; no longer LINE_IN.3, U$6.COM1
- net N$12: now also FB3.2, REL1A.COM; no longer HEADPHONES.5, U$3.COM1
- net N$14: now also FB6.2, REL1A.NC, REL1B.NO; no longer LINE_IN.5, U$3.NC1, U$3.NO2
- net N$2: now also REL3A.NO; no longer U$6.NO1
- net N$3: now also FB1.2, REL2A.NO, REL3A.NC; no longer HEADPHONES.3, U$4.NO1, U$6.NC1
- net N$4: now also FB2.2, REL2B.NO, REL3B.NC; no longer HEADPHONES.2, U$4.NO2, U$6.NC2
- net N$5: now also FB5.2, REL3B.COM; no longer LINE_IN.2, U$6.COM2
- net N$6: now also REL3B.NO; no longer U$6.NO2
Other:
- note added: "TODO fixed boot mode"
- note added: "TODO hook up to GPIO (with jumper to power line)"
- note removed: "Audio"
- note removed: "TODO check this"
- note removed: "TODO connect coils to power or GPIO or choice jumpers"
- note removed: "TODO ferrite beads HZ0805D152R-10"
- moved on the sheet: C27, C28, HEADPHONES, LINE_IN, R3, R4, R5, R6, R7, R8
